Commit message: gazebo simulation

File: description/robot.urdf.xacro (robot description, xacro)
@@ -2,3 +2,4 @@
 <robot xmlns:xacro="http://www.ros.org/wiki/xacro"  name="robot">
     <xacro:include filename="robot_core.urdf.xacro" />
+    <xacro:include filename="gazebo_control.urdf.xacro" />
 </robot>

File: description/robot_core.urdf.xacro (robot description, xacro)
@@ -2,5 +2,5 @@
 <robot xmlns:xacro="http://www.ros.org/wiki/xacro">
     <xacro:include filename="inertial_macros.urdf.xacro" />
-   <material name="white">
+    <material name="white">
         <color rgba="1 1 1 1"/>
     </material>
@@ -40,5 +40,5 @@
         </xacro:inertial_box>
     </link>
-     <!-- LEFT WHEEL -->
+    <!-- LEFT WHEEL -->
     <joint name="left_wheel_joint" type="continuous">
         <parent link="base_link"/>
@@ -46,4 +46,5 @@
         <origin xyz="0 0.175 0" rpy="-${pi/2} 0 0"/>
         <axis xyz="0 0 1"/>
+        <limit effort="0.05" velocity="10.0"/>
     </joint>
     <link name="left_wheel">
@@ -56,5 +57,5 @@
         <collision>
             <geometry>
-                <cylinder length="0.04" radius="0.05" />
+                <sphere radius="0.05" />
             </geometry>
         </collision>
@@ -69,4 +70,5 @@
         <origin xyz="0 -0.175 0" rpy="${pi/2} 0 0"/>
         <axis xyz="0 0 -1"/>
+        <limit effort="0.05" velocity="10.0"/>
     </joint>
     <link name="right_wheel">
@@ -79,5 +81,5 @@
         <collision>
             <geometry>
-                <cylinder length="0.04" radius="0.05" />
+                <sphere radius="0.05" />
             </geometry>
         </collision>
@@ -104,7 +106,11 @@
             </geometry>
         </collision>
-         <xacro:inertial_sphere mass="0.1" radius="0.05">
+        <xacro:inertial_sphere mass="0.1" radius="0.05">
             <origin xyz="0 0 0" rpy="0 0 0"/>
         </xacro:inertial_sphere>
     </link>
+    <gazebo reference="caster_wheel">
+        <mu1 value="0.0"/>
+        <mu2 value="0.0"/>
+    </gazebo>
 </robot>
